File: TFG-Brushless-ESC/Half-Bridge.kicad_sch (KiCad schematic)
At the start: 28 parts, among them Q5 TK58E06N1, Q6 TK58E06N1, U8 IR2101, U9 INA180A3

Commit message: mas traducciones
Other:
- note added: "Shunt (medida)"
- note removed: "Shunt corriente"
Changed lines of the file:
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@@
 		)
 	)
-	(text "Shunt corriente"
+	(text "Shunt (medida)"
 		(exclude_from_sim no)
 		(at 154.305 108.585 0)
