File: TFG-Brushless-ESC/TFG-Brushless-ESC.kicad_sch (KiCad schematic)
At the start: 72 parts, among them J2 USB C Receptacle, J3 HALL SENSORS, J4 SWD-I2C, J5 24V IN, Q7 DMG3402L, SW1 BOOT0, SW2 NRST, U1 LM317L_SOT-89, U10 ADS7830, U2 LM317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

Commit message: mas traducciones
Other:
- note added: "- 1 condensador por pin VDD. - Mantener lo más cerca posible del IC. - Tamaño máximo: 0603"
- note added: "Condensador electrolítico extra de 220u si el regulador no está próximo al raíl de 5V"
- note removed: "- 1 capacitor per VDD pin. - Keep as close as possible to the IC. - Maximum size: 0603"
- note removed: "Extra 220u electrolytic if not close to 5V supply"
Changed lines of the file:
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@@
 	)
 	(junction
-		(at 95.25 36.195)
-		(diameter 0)
-		(color 0 0 0 0)
-	)
-	(junction
 		(at 34.29 90.805)
 		(diameter 0)
@@
 	(wire
 		(pts
-			(xy 103.505 36.195) (xy 95.25 36.195)
-		)
-		(stroke
-			(width 0)
-			(type default)
-		)
-	)
-	(wire
-		(pts
 			(xy 169.545 81.915) (xy 170.815 81.915)
 		)
@@
 		)
 	)
-	(text "- 1 capacitor per VDD pin.\n- Keep as close as possible\n  to the IC.\n- Maximum size: 0603"
+	(text "- 1 condensador por pin VDD.\n- Mantener lo más cerca posible del IC.\n- Tamaño máximo: 0603"
 		(exclude_from_sim no)
-		(at 243.205 29.21 0)
+		(at 237.49 26.035 0)
 		(effects
 			(font
@@
 		)
 	)
-	(text "Extra 220u\nelectrolytic if\nnot close to\n5V supply"
+	(text "Condensador\nelectrolítico\nextra de 220u\nsi el regulador\nno está próximo\nal raíl de 5V"
 		(exclude_from_sim no)
-		(at 74.295 40.005 0)
+		(at 74.295 40.64 0)
 		(effects
 			(font
@@
 	)
 	(label "V_DIV_3"
-		(at 103.505 36.195 180)
+		(at 93.98 36.195 180)
 		(effects
 			(font
@@
 	(symbol
 		(lib_id "Graphic:SYM_Arrow_Normal")
-		(at 74.295 31.115 90)
+		(at 74.295 30.48 90)
 		(unit 1)
 		(exclude_from_sim yes)
@@
 		(fields_autoplaced yes)
 		(property "Reference" "#SYM1"
-			(at 72.771 31.115 0)
+			(at 72.771 30.48 0)
 			(effects
 				(font
@@
 		)
 		(property "Value" "SYM_Arrow_Normal"
-			(at 75.565 30.861 0)
+			(at 75.565 30.226 0)
 			(effects
 				(font
@@
 		)
 		(property "Footprint" ""
-			(at 74.295 31.115 0)
+			(at 74.295 30.48 0)
 			(effects
 				(font
@@
 		)
 		(property "Datasheet" "~"
-			(at 74.295 31.115 0)
+			(at 74.295 30.48 0)
 			(effects
 				(font
@@
 		)
 		(property "Description" "Filled arrow, 200mil"
-			(at 74.295 31.115 0)
+			(at 74.295 30.48 0)
 			(effects
 				(font
